Commit message: Add trailer_body file (copy of mpo500 body)

File: robots/mpo_500/mpo_500.urdf.xacro (robot description, xacro)
@@ -17,4 +17,7 @@
   <-->
   <!-- <xacro:include filename="$(find neo_simulation)/robots/mpo_500/xacros/camera.xacro" />  -->
+  <!--TRAILER-->
+  <!-- TRAILER BODY -->
+  <xacro:include filename="$(find neo_simulation)/robots/mpo_500/xacros/mpo_500_trailer_body.xacro" />
   <link name="base_link" />
   <!-- Base link macro -->
@@ -22,4 +25,8 @@
     <origin xyz="0 0 0" rpy="0 0 0" />
   </xacro:mpo_500_base>
+  <!-- Base link macro -->
+  <xacro:mpo_500_trailer_base name="trailer_footprint" parent="base_footprint">
+    <origin xyz="-1 0 0" rpy="0 0 0" />
+  </xacro:mpo_500_trailer_base>
   <!-- Wheel Macro -->
   <xacro:omni_wheel_250 name="mpo_500_omni_wheel_front_left" parent="base_footprint">

Commit message: Add parameter to change properties of trailer body

File: robots/mpo_500/mpo_500.urdf.xacro (robot description, xacro)
@@ -20,4 +20,5 @@
   <!-- TRAILER BODY -->
   <xacro:include filename="$(find neo_simulation)/robots/mpo_500/xacros/mpo_500_trailer_body.xacro" />
+  <xacro:include filename="$(find neo_simulation)/robots/mpo_500/xacros/mpo_500_trailer_parameter.xacro" />
   <link name="base_link" />
   <!-- Base link macro -->
@@ -26,6 +27,7 @@
   </xacro:mpo_500_base>
   <!-- Base link macro -->
-  <xacro:mpo_500_trailer_base name="trailer_footprint" parent="base_footprint">
+  <xacro:mpo_500_trailer_base name="trailer_footprint" parent="base_footprint" >
     <origin xyz="-1 0 0" rpy="0 0 0" />
+    <!--xacro:property name="x_length_chassis_trailer" value="2.0" /-->
   </xacro:mpo_500_trailer_base>
   <!-- Wheel Macro -->

File: robots/mpo_500/xacros/mpo_500_trailer_body.xacro (robot description, xacro)
@@ -1,4 +1,6 @@
 <?xml version="1.0"?>
 <robot xmlns:xacro="http://www.ros.org/wiki/xacro" name="mpo_500">
+  <!--xacro:include filename="$(find PeTRA)/neo_simulation/robots/mpo_500/xacros/mpo_500_trailer_parameter.xacro"/-->
+  <xacro:include filename="$(find neo_simulation)/robots/mpo_500/xacros/mpo_500_trailer_parameter.xacro" />
   <xacro:macro name="mpo_500_trailer_base" params="name parent *origin">
     <joint name="${name}_joint" type="revolute">
@@ -20,5 +22,5 @@
         <origin xyz="-0.5 0. 0.25" rpy="-1.571 0 1.571" />
         <geometry>
-          <box size="1 0.25 1.5"/>
+          <box size="${x_length_chassis_trailer} ${y_length_chassis_trailer} ${z_length_chassis_trailer}"/>
         </geometry>
       </visual>
@@ -26,5 +28,5 @@
         <origin xyz="-0.5 0. 0.25" rpy="-1.571 0 1.571" />
         <geometry>
-          <box size="1 0.25 1.5"/>
+          <box size="${x_length_chassis_trailer} ${y_length_chassis_trailer} ${z_length_chassis_trailer}"/>
         </geometry>
       </collision>

File: robots/mpo_500/xacros/mpo_500_trailer_parameter.xacro (robot description, xacro)
@@ -1,15 +1,15 @@
 <?xml version="1.0"?>
 <robot xmlns:xacro="http://ww.ros.org/wiki/xacro">
-    <!-- Define parameter for the differntial drive robot -->
+    <!-- Define parameter for the trailer -->
     <!-- Parameter for the chassis, size [m] and mass [kg] -->
-    <xacro:property name="x_chassis" value="0.5" />
-    <xacro:property name="y_chassis" value="0.3" />
-    <xacro:property name="z_chassis" value="0.15" />
-    <xacro:property name="m_chassis" value="10.0" />
+    <xacro:property name="x_length_chassis_trailer" value="1.0" />
+    <xacro:property name="y_length_chassis_trailer" value="0.25" />
+    <xacro:property name="z_length_chassis_trailer" value="1.5" />
+    <xacro:property name="mass_chassis_trailer" value="64.0" />
     <!-- Parameter for the wheels, radius [m], height [m], mass [kg], torque[Nm], wheelbase [m] -->
-    <xacro:property name="r_wheel" value="0.1075" />
-    <xacro:property name="h_wheel" value="0.03" />
-    <xacro:property name="m_wheel" value="3.0" />
-    <xacro:property name="torque_wheel" value="10" />
+    <xacro:property name="radius_wheel_trailer" value="0.1075" />
+    <xacro:property name="height_wheel_trailer" value="0.03" />
+    <xacro:property name="mass_wheel_trailer" value="3.0" />
+    <xacro:property name="torque_wheel_trailer" value="10" />
     <xacro:property name="L_wheel" value="0.1788" />
 </robot>

Commit message: Add trailer body origin variable

File: robots/mpo_500/mpo_500.urdf.xacro (robot description, xacro)
@@ -20,15 +20,54 @@
   <!-- TRAILER BODY -->
   <xacro:include filename="$(find neo_simulation)/robots/mpo_500/xacros/mpo_500_trailer_body.xacro" />
+  <!-- TRAILER PARAMETER-->
   <xacro:include filename="$(find neo_simulation)/robots/mpo_500/xacros/mpo_500_trailer_parameter.xacro" />
+  <!-- TRAILER WHEEL-->
+  <xacro:include filename="$(find neo_simulation)/robots/mpo_500/xacros/mpo_500_trailer_wheel.xacro" />
   <link name="base_link" />
+  <!-- TRAILER START-->
+  <!-- Base link macro -->
+  <xacro:mpo_500_trailer_base name="trailer_footprint" parent="base_footprint" >
+    <origin xyz="0 0 0" rpy="0 0 0" />
+  </xacro:mpo_500_trailer_base>
+  <!-- TRAILER WHEEL macro-->
+  <xacro:trailer_wheel name="mpo_500_trailer_wheel_front_left" parent="trailer_footprint">
+    <origin xyz="0
+    0
+    0"
+    rpy="0 0 0" />
+  </xacro:trailer_wheel>
+  <xacro:trailer_wheel name="mpo_500_trailer_wheel_middle_left" parent="trailer_footprint">
+    <origin xyz="-0.75
+    0
+    0"
+    rpy="0 0 0" />
+  </xacro:trailer_wheel>
+  <xacro:trailer_wheel name="mpo_500_trailer_wheel_back_left" parent="trailer_footprint">
+    <origin xyz="-1.5
+    0
+    0"
+    rpy="0 0 0" />
+  </xacro:trailer_wheel>
+   <!--
+  <xacro:trailer_wheel name="mpo_500_trailer_wheel_middle_left" parent="trailer_footprint">
+    <origin xyz="${x_length_chassis_trailer}
+    radius_wheel_trailer/2-y_length_chassis_trailer/2
+     -z_length_chassis_trailer/4" rpy="0 0 0" />
+  </xacro:trailer_wheel>
+-->
+ <!--
+  <xacro:trailer_wheel name="mpo_500_trailer_wheel_back_left" parent="trailer_footprint">
+    <origin xyz="${radius_wheel_trailer/x_length_chassis_trailer/2}
+    radius_wheel_trailer/2-y_length_chassis_trailer/2 -z_length_chassis_trailer/4" rpy="0 0 0" />
+  </xacro:trailer_wheel>
+    -->
+<!-- ${-x_length_chassis_trailer/4}-->
+<!-- ${y_length_chassis_trailer/2+height_wheel_trailer}-->
+<!-- ${radius_wheel_trailer/2-z_length_chassis_trailer/2}-->
+  <!-- TRAILER END-->
   <!-- Base link macro -->
   <xacro:mpo_500_base name="base_footprint" parent="base_link">
     <origin xyz="0 0 0" rpy="0 0 0" />
   </xacro:mpo_500_base>
-  <!-- Base link macro -->
-  <xacro:mpo_500_trailer_base name="trailer_footprint" parent="base_footprint" >
-    <origin xyz="-1 0 0" rpy="0 0 0" />
-    <!--xacro:property name="x_length_chassis_trailer" value="2.0" /-->
-  </xacro:mpo_500_trailer_base>
   <!-- Wheel Macro -->
   <xacro:omni_wheel_250 name="mpo_500_omni_wheel_front_left" parent="base_footprint">

File: robots/mpo_500/xacros/mpo_500_trailer_body.xacro (robot description, xacro)
@@ -20,5 +20,5 @@
       </inertial>
       <visual>
-        <origin xyz="-0.5 0. 0.25" rpy="-1.571 0 1.571" />
+        <origin xyz="${x_origin_chassis_trailer} ${y_origin_chassis_trailer} ${z_origin_chassis_trailer}" rpy="-1.571 0 1.571" />
         <geometry>
           <box size="${x_length_chassis_trailer} ${y_length_chassis_trailer} ${z_length_chassis_trailer}"/>
@@ -26,5 +26,5 @@
       </visual>
       <collision>
-        <origin xyz="-0.5 0. 0.25" rpy="-1.571 0 1.571" />
+        <origin xyz="${x_origin_chassis_trailer} ${y_origin_chassis_trailer} ${z_origin_chassis_trailer}" rpy="-1.571 0 1.571" />
         <geometry>
           <box size="${x_length_chassis_trailer} ${y_length_chassis_trailer} ${z_length_chassis_trailer}"/>

File: robots/mpo_500/xacros/mpo_500_trailer_parameter.xacro (robot description, xacro)
@@ -7,7 +7,11 @@
     <xacro:property name="z_length_chassis_trailer" value="1.5" />
     <xacro:property name="mass_chassis_trailer" value="64.0" />
+    <!-- Parameter for the origin of the chassis -->
+    <xacro:property name="x_origin_chassis_trailer" value="-1.5" />
+    <xacro:property name="y_origin_chassis_trailer" value="0" />
+    <xacro:property name="z_origin_chassis_trailer" value="0.25" />
     <!-- Parameter for the wheels, radius [m], height [m], mass [kg], torque[Nm], wheelbase [m] -->
-    <xacro:property name="radius_wheel_trailer" value="0.1075" />
-    <xacro:property name="height_wheel_trailer" value="0.03" />
+    <xacro:property name="radius_wheel_trailer" value="0.126" />
+    <xacro:property name="height_wheel_trailer" value="0.110" />
     <xacro:property name="mass_wheel_trailer" value="3.0" />
     <xacro:property name="torque_wheel_trailer" value="10" />

Commit message: Fix oriantation of x y z of trailer chassis

File: robots/mpo_500/mpo_500.urdf.xacro (robot description, xacro)
@@ -32,34 +32,22 @@
   <!-- TRAILER WHEEL macro-->
   <xacro:trailer_wheel name="mpo_500_trailer_wheel_front_left" parent="trailer_footprint">
-    <origin xyz="0
-    0
-    0"
-    rpy="0 0 0" />
+    <origin xyz="${x_origin_chassis_trailer-x_length_chassis_trailer/2+radius_wheel_trailer} 0.28 0.13" rpy="0 0 0" />
   </xacro:trailer_wheel>
-  <xacro:trailer_wheel name="mpo_500_trailer_wheel_middle_left" parent="trailer_footprint">
-    <origin xyz="-0.75
-    0
-    0"
-    rpy="0 0 0" />
+  <xacro:trailer_wheel name="mpo_500_trailer_wheel_front_right" parent="trailer_footprint">
+    <origin xyz="0.25 -0.28 0.13" rpy="0 0 3.14" />
   </xacro:trailer_wheel>
   <xacro:trailer_wheel name="mpo_500_trailer_wheel_back_left" parent="trailer_footprint">
-    <origin xyz="-1.5
-    0
-    0"
+    <origin xyz="-0.25 0.28 0.13" rpy="0 0 0" />
+  </xacro:trailer_wheel>
+  <xacro:trailer_wheel name="mpo_500_trailer_wheel_back_right" parent="trailer_footprint">
+    <origin xyz="-0.25 -0.28 0.13" rpy="0 0 3.14" />
+  </xacro:trailer_wheel>
+  <!--
+  <xacro:trailer_wheel name="mpo_500_trailer_wheel_front_left" parent="trailer_footprint">
+    <origin xyz="${x_origin_chassis_trailer+x_length_chassis_trailer/2+radius_wheel_trailer}
+    ${y_origin_chassis_trailer+x_length_chassis_trailer}
+    ${z_origin_chassis_trailer}"
     rpy="0 0 0" />
-  </xacro:trailer_wheel>
-   <!--
-  <xacro:trailer_wheel name="mpo_500_trailer_wheel_middle_left" parent="trailer_footprint">
-    <origin xyz="${x_length_chassis_trailer}
-    radius_wheel_trailer/2-y_length_chassis_trailer/2
-     -z_length_chassis_trailer/4" rpy="0 0 0" />
-  </xacro:trailer_wheel>
--->
- <!--
-  <xacro:trailer_wheel name="mpo_500_trailer_wheel_back_left" parent="trailer_footprint">
-    <origin xyz="${radius_wheel_trailer/x_length_chassis_trailer/2}
-    radius_wheel_trailer/2-y_length_chassis_trailer/2 -z_length_chassis_trailer/4" rpy="0 0 0" />
-  </xacro:trailer_wheel>
-    -->
+  </xacro:trailer_wheel> -->
 <!-- ${-x_length_chassis_trailer/4}-->
 <!-- ${y_length_chassis_trailer/2+height_wheel_trailer}-->

File: robots/mpo_500/xacros/mpo_500_trailer_body.xacro (robot description, xacro)
@@ -22,5 +22,5 @@
         <origin xyz="${x_origin_chassis_trailer} ${y_origin_chassis_trailer} ${z_origin_chassis_trailer}" rpy="-1.571 0 1.571" />
         <geometry>
-          <box size="${x_length_chassis_trailer} ${y_length_chassis_trailer} ${z_length_chassis_trailer}"/>
+          <box size="${y_length_chassis_trailer} ${z_length_chassis_trailer} ${x_length_chassis_trailer}"/>
         </geometry>
       </visual>
@@ -28,5 +28,5 @@
         <origin xyz="${x_origin_chassis_trailer} ${y_origin_chassis_trailer} ${z_origin_chassis_trailer}" rpy="-1.571 0 1.571" />
         <geometry>
-          <box size="${x_length_chassis_trailer} ${y_length_chassis_trailer} ${z_length_chassis_trailer}"/>
+          <box size="${y_length_chassis_trailer} ${z_length_chassis_trailer} ${x_length_chassis_trailer}"/>
         </geometry>
       </collision>

File: robots/mpo_500/xacros/mpo_500_trailer_parameter.xacro (robot description, xacro)
@@ -3,12 +3,14 @@
     <!-- Define parameter for the trailer -->
     <!-- Parameter for the chassis, size [m] and mass [kg] -->
-    <xacro:property name="x_length_chassis_trailer" value="1.0" />
-    <xacro:property name="y_length_chassis_trailer" value="0.25" />
-    <xacro:property name="z_length_chassis_trailer" value="1.5" />
+    <xacro:property name="x_length_chassis_trailer" value="1.5" />
+    <xacro:property name="y_length_chassis_trailer" value="1.0" />
+    <xacro:property name="z_length_chassis_trailer" value="0.25" />
     <xacro:property name="mass_chassis_trailer" value="64.0" />
     <!-- Parameter for the origin of the chassis -->
     <xacro:property name="x_origin_chassis_trailer" value="-1.5" />
     <xacro:property name="y_origin_chassis_trailer" value="0" />
-    <xacro:property name="z_origin_chassis_trailer" value="0.25" />
+    <xacro:property name="z_origin_chassis_trailer" value="0.4" />
+    <!-- Parameter for the origin of trailer_wheel_front_left -->
+    <xacro:property name="x_origin_trailer_wheel_front_left" value="-1.5" />
     <!-- Parameter for the wheels, radius [m], height [m], mass [kg], torque[Nm], wheelbase [m] -->
     <xacro:property name="radius_wheel_trailer" value="0.126" />

File: robots/mpo_500/xacros/mpo_500_trailer_wheel.xacro (robot description, xacro)
@@ -22,5 +22,5 @@
     </inertial>
     <visual>
-     <origin xyz="0 0 0" rpy="0 0 0"/>
+     <origin xyz="0 0 0" rpy="0 1.57 1.57"/>
      <geometry>
       <cylinder radius="${radius_wheel_trailer}" length="${height_wheel_trailer}"/>

Commit message: Make wheels position dependend on chassis values

File: robots/mpo_500/mpo_500.urdf.xacro (robot description, xacro)
@@ -30,16 +30,22 @@
     <origin xyz="0 0 0" rpy="0 0 0" />
   </xacro:mpo_500_trailer_base>
-  <!-- TRAILER WHEEL macro-->
+  <!-- TRAILER WHEEL macro: Wheels depend on the height and length of the chassis. Wheels depnd not on the height of the chassis.-->
   <xacro:trailer_wheel name="mpo_500_trailer_wheel_front_left" parent="trailer_footprint">
-    <origin xyz="${x_origin_chassis_trailer-x_length_chassis_trailer/2+radius_wheel_trailer} 0.28 0.13" rpy="0 0 0" />
+    <origin xyz="${x_origin_chassis_trailer-x_length_chassis_trailer/2+radius_wheel_trailer} ${y_length_chassis_trailer/2-height_wheel_trailer/2} ${radius_wheel_trailer}" rpy="0 0 0" />
   </xacro:trailer_wheel>
   <xacro:trailer_wheel name="mpo_500_trailer_wheel_front_right" parent="trailer_footprint">
-    <origin xyz="0.25 -0.28 0.13" rpy="0 0 3.14" />
+    <origin xyz="${x_origin_chassis_trailer-x_length_chassis_trailer/2+radius_wheel_trailer} ${-y_length_chassis_trailer/2+height_wheel_trailer/2} ${radius_wheel_trailer}" rpy="0 0 3.14" />
+  </xacro:trailer_wheel>
+  <xacro:trailer_wheel name="mpo_500_trailer_wheel_middle_left" parent="trailer_footprint">
+    <origin xyz="${x_origin_chassis_trailer} ${y_length_chassis_trailer/2-height_wheel_trailer/2} ${radius_wheel_trailer}" rpy="0 0 0" />
+  </xacro:trailer_wheel>
+  <xacro:trailer_wheel name="mpo_500_trailer_wheel_middle_right" parent="trailer_footprint">
+    <origin xyz="${x_origin_chassis_trailer} ${-y_length_chassis_trailer/2+height_wheel_trailer/2} ${radius_wheel_trailer}" rpy="0 0 3.14" />
   </xacro:trailer_wheel>
   <xacro:trailer_wheel name="mpo_500_trailer_wheel_back_left" parent="trailer_footprint">
-    <origin xyz="-0.25 0.28 0.13" rpy="0 0 0" />
+    <origin xyz="${x_origin_chassis_trailer+x_length_chassis_trailer/2-radius_wheel_trailer} ${y_length_chassis_trailer/2-height_wheel_trailer/2} ${radius_wheel_trailer}" rpy="0 0 0" />
   </xacro:trailer_wheel>
   <xacro:trailer_wheel name="mpo_500_trailer_wheel_back_right" parent="trailer_footprint">
-    <origin xyz="-0.25 -0.28 0.13" rpy="0 0 3.14" />
+    <origin xyz="${x_origin_chassis_trailer+x_length_chassis_trailer/2-radius_wheel_trailer} ${-y_length_chassis_trailer/2+height_wheel_trailer/2} ${radius_wheel_trailer}" rpy="0 0 3.14" />
   </xacro:trailer_wheel>
   <!--

Commit message: Add Slip to the wheel

File: robots/mpo_500/mpo_500.urdf.xacro (robot description, xacro)
@@ -30,22 +30,82 @@
     <origin xyz="0 0 0" rpy="0 0 0" />
   </xacro:mpo_500_trailer_base>
-  <!-- TRAILER WHEEL macro: Wheels depend on the height and length of the chassis. Wheels depnd not on the height of the chassis.-->
+  <!-- TRAILER WHEEL macro: Wheels depend on the height and length of the chassis. Wheels depend not on the height of the chassis.-->
   <xacro:trailer_wheel name="mpo_500_trailer_wheel_front_left" parent="trailer_footprint">
     <origin xyz="${x_origin_chassis_trailer-x_length_chassis_trailer/2+radius_wheel_trailer} ${y_length_chassis_trailer/2-height_wheel_trailer/2} ${radius_wheel_trailer}" rpy="0 0 0" />
+    <surface>
+      <friction>
+          <ode>
+              <mu>0</mu>
+              <mu2>0</mu2>
+              <slip1>1.0</slip1>
+              <slip2>1.0</slip2>
+          </ode>
+      </friction>
+    </surface>
   </xacro:trailer_wheel>
   <xacro:trailer_wheel name="mpo_500_trailer_wheel_front_right" parent="trailer_footprint">
     <origin xyz="${x_origin_chassis_trailer-x_length_chassis_trailer/2+radius_wheel_trailer} ${-y_length_chassis_trailer/2+height_wheel_trailer/2} ${radius_wheel_trailer}" rpy="0 0 3.14" />
+    <surface>
+      <friction>
+          <ode>
+              <mu>0</mu>
+              <mu2>0</mu2>
+              <slip1>1.0</slip1>
+              <slip2>1.0</slip2>
+          </ode>
+      </friction>
+    </surface>
   </xacro:trailer_wheel>
   <xacro:trailer_wheel name="mpo_500_trailer_wheel_middle_left" parent="trailer_footprint">
     <origin xyz="${x_origin_chassis_trailer} ${y_length_chassis_trailer/2-height_wheel_trailer/2} ${radius_wheel_trailer}" rpy="0 0 0" />
+    <surface>
+      <friction>
+          <ode>
+              <mu>1</mu>
+              <mu2>1</mu2>
+              <slip1>0.0</slip1>
+              <slip2>0.0</slip2>
+          </ode>
+      </friction>
+    </surface>
   </xacro:trailer_wheel>
   <xacro:trailer_wheel name="mpo_500_trailer_wheel_middle_right" parent="trailer_footprint">
     <origin xyz="${x_origin_chassis_trailer} ${-y_length_chassis_trailer/2+height_wheel_trailer/2} ${radius_wheel_trailer}" rpy="0 0 3.14" />
+    <surface>
+      <friction>
+          <ode>
+              <mu>1</mu>
+              <mu2>1</mu2>
+              <slip1>0.0</slip1>
+              <slip2>0.0</slip2>
+          </ode>
+      </friction>
+    </surface>
   </xacro:trailer_wheel>
   <xacro:trailer_wheel name="mpo_500_trailer_wheel_back_left" parent="trailer_footprint">
     <origin xyz="${x_origin_chassis_trailer+x_length_chassis_trailer/2-radius_wheel_trailer} ${y_length_chassis_trailer/2-height_wheel_trailer/2} ${radius_wheel_trailer}" rpy="0 0 0" />
+    <surface>
+      <friction>
+          <ode>
+              <mu>0</mu>
+              <mu2>0</mu2>
+              <slip1>1.0</slip1>
+              <slip2>1.0</slip2>
+          </ode>
+      </friction>
+    </surface>
   </xacro:trailer_wheel>
   <xacro:trailer_wheel name="mpo_500_trailer_wheel_back_right" parent="trailer_footprint">
     <origin xyz="${x_origin_chassis_trailer+x_length_chassis_trailer/2-radius_wheel_trailer} ${-y_length_chassis_trailer/2+height_wheel_trailer/2} ${radius_wheel_trailer}" rpy="0 0 3.14" />
+    <surface>
+      <friction>
+          <ode>
+              <mu>0</mu>
+              <mu2>0</mu2>
+              <slip1>1.0</slip1>
+              <slip2>1.0</slip2>
+          </ode>
+      </friction>
+    </surface>
   </xacro:trailer_wheel>
   <!--

File: robots/mpo_500/xacros/mpo_500_trailer_wheel.xacro (robot description, xacro)
@@ -3,5 +3,5 @@
   <!-- Include parameter for trailer-->
   <xacro:include filename="$(find neo_simulation)/robots/mpo_500/xacros/mpo_500_trailer_parameter.xacro" />
-  <xacro:macro name="trailer_wheel" params="name parent *origin">
+  <xacro:macro name="trailer_wheel" params="name parent *origin *surface">
    <joint name="${name}_joint" type="revolute">
     <xacro:insert_block name="origin" />
@@ -34,4 +34,5 @@
         <!-- <mesh filename="package://neo_simulation/robots/mpo_500/meshes/MPO-500-WHEEL.dae" scale="0.001 0.001 0.001"/> -->
        <!-- <cylinder radius="0.126" length="0.110"/> -->
+       <xacro:insert_block name="surface" />
      </geometry>
     </collision>
